File: EAGLE/src/Wooby.sch (EAGLE design)
At the start: 18 parts, among them J2 691210910002, J5 691210910002, U1 GY-521MPU6050

Commit message: Release version 1 just before shipping!
Other:
- note added: "SCL(GPIO22)"
- note added: "SDA(GPIO21)"
Changed lines of the file:
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@@
 <text x="2.54" y="73.66" size="1.778" layer="91">White</text>
 <text x="2.54" y="83.82" size="1.778" layer="91">Red</text>
+<text x="-5.08" y="-15.24" size="1.778" layer="91">SCL(GPIO22)</text>
+<text x="-5.08" y="-10.16" size="1.778" layer="91">SDA(GPIO21)</text>
 </plain>
 <instances>
