File: EAGLE/src/Wooby.brd (EAGLE design)
At the start: 170 x 80 mm, 30 parts, among them J1 691210910002, J2 691210910002, J3 691210910002, J4 691210910002, J5 691210910002

Commit message: Lady D Version
Parts:
- removed CELL, CELL1, CELL2, CELL3, J1, J2, J3, J4, J5: 691210910002, 691210910002:691210910002
- added SV1, SV2, SV3, SV4: (no value), con-lstb:MA04-1
- LCD: value 691210910002 -> (none); device 691210910002:691210910002 -> con-lstb:MA04-1
- moved ON_BTN 36.9 mm to (12.0, 58.0), turned to 90 degrees
- moved LCD 6.00 mm to (87.0, 70.0), turned to 0 degrees
- moved SM4 5.30 mm to (140.0, 13.0)
- moved SM2 5.05 mm to (140.0, 67.0)
- moved U$3 5.00 mm to (120.0, 65.4)
- moved ESP32-DEVKITC 3.00 mm to (102.0, 40.0)
- moved SM1 1.48 mm to (35.0, 13.0)
- moved U$2 1.00 mm to (86.0, 65.4)
- moved SM3 0.96 mm to (35.0, 67.0)
Connections:
- net +3V3: now also LCD.3; no longer LCD.1
- net GND: now also LCD.4; no longer LCD.2
- net N$1: now also SV1.3; no longer CELL.1
- net N$13: now also SV4.4; no longer CELL3.2
- net N$14: now also SV4.3; no longer CELL3.1
- net N$15: now also SV4.2; no longer J4.2
- net N$16: now also SV4.1; no longer J4.1
- net N$17: now also SV3.4; no longer CELL2.2
- net N$18: now also SV3.3; no longer CELL2.1
- net N$19: now also SV3.2; no longer J3.2
- net N$2: now also SV1.4; no longer CELL.2
- net N$20: now also SV3.1; no longer J3.1
- net N$21: now also SV2.4; no longer CELL1.2
- net N$22: now also SV2.3; no longer CELL1.1
- net N$23: now also SV2.2; no longer J1.2
- net N$24: now also SV2.1; no longer J1.1
- net N$3: now also SV1.1; no longer J5.1
- net N$4: now also SV1.2; no longer J5.2
- net N$6: now also LCD.2; no longer J2.2
- net N$7: now also LCD.1; no longer J2.1
Routing:
- net N$52: track 5.64 -> 46.8 mm
- net N$26: track 3.73 -> 34.0 mm
- net N$7: track 60.9 -> 74.3 mm
- net N$9: track 89.0 -> 102.3 mm
- net N$6: track 44.5 -> 50.6 mm
- net N$10: track 131.9 -> 137.4 mm
- net N$8: track 248.3 -> 253.7 mm
- net N$5: track 53.6 -> 57.3 mm
- net N$16: track 11.0 -> 7.52 mm
- net N$15: track 11.0 -> 7.52 mm
- net N$22: track 10.9 -> 7.52 mm
- net N$21: track 10.9 -> 7.52 mm
- net N$24: track 10.6 -> 7.52 mm
- net N$13: track 10.5 -> 7.52 mm
- net N$14: track 10.5 -> 7.52 mm
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Other:
- board text added: "100nF"
- board text added: "47uF"
- board text added: "LCD"
- board text added: "Lady D Version"
- board text added: "SCL"
- board text added: "SDA"
